Commit message: added front left wheel

File: description/robot_core.xacro (robot description, xacro)
@@ -1,7 +1,40 @@
 <?xml version="1.0"?>
 <robot xmlns:xacro="http://www.ros.org/wiki/xacro">
-    <!-- joints go here -->
+    <!-- links and joints go here -->
     <!-- The rest of the robot can be described from base_link, which is the centre point of the four driving wheels -->
     <link name="base_link">
     </link>
+    <!-- chassis joint goes here. It connects chassis to base_link via fixed joint -->
+    <joint name="chassis_joint" type="fixed">
+        <parent link="base_link"/>
+        <child link="chassis"/>
+        <origin xyz="0 0 0"/>
+    </joint>
+    <!-- chassis description goes here. It describes the chassis of robocock which is a 54cm x 54cm x 150cm box -->
+    <link name="chassis">
+        <visual>
+            <!-- by default, the origin is centred around the link origin, so offset it by half the height -->
+            <origin xyz="0 0 0.75" rpy="0 0 0"/>
+            <geometry>
+                <box size="0.54 0.54 1.5"/>
+            </geometry>
+            <material name="white"/>
+        </visual>
+    </link>
+    <!-- FRONT LEFT WHEEL AKA wheel_1 -->
+    <joint name="wheel_1_joint" type="continuous">
+        <parent link="base_link"/>
+        <child link="wheel_1"/>
+        <origin xyz="0 0.285 0" rpy="-${pi/2} 0 0"/>
+        <axis xyz="0 0 1"/>
+    </joint>
+    <link name="wheel_1">
+        <visual>
+            <geometry>
+                <!-- width of wheel assumed to be 3 cm -->
+                <cylinder length="0.03" radius="0.05"/>
+            </geometry>
+            <material name="blue"/>
+        </visual>
+    </link>
 </robot>

Commit message: wheel test

File: description/robot_core.xacro (robot description, xacro)
@@ -32,6 +32,5 @@
         <visual>
             <geometry>
-                <!-- width of wheel assumed to be 3 cm -->
-                <cylinder length="0.03" radius="0.05"/>
+                <cylinder length="0.038" radius="0.05"/>
             </geometry>
             <material name="blue"/>

Commit message: all wheels defined and functional independently

File: description/robot_core.xacro (robot description, xacro)
@@ -26,5 +26,5 @@
         <parent link="base_link"/>
         <child link="wheel_1"/>
-        <origin xyz="0 0.285 0" rpy="-${pi/2} 0 0"/>
+        <origin xyz="0.1575 0.1575 0" rpy="-${pi/2} 0 -${pi/4}"/>
         <axis xyz="0 0 1"/>
     </joint>
@@ -32,5 +32,50 @@
         <visual>
             <geometry>
-                <cylinder length="0.038" radius="0.05"/>
+                <cylinder length="0.038" radius="0.05" />/>
+            </geometry>
+            <material name="blue"/>
+        </visual>
+    </link>
+    <!-- FRONT RIGHT WHEEL AKA wheel_2 -->
+    <joint name="wheel_2_joint" type="continuous">
+        <parent link="base_link"/>
+        <child link="wheel_2"/>
+        <origin xyz="0.1575 -0.1575 0" rpy="${pi/2} 0 ${pi/4}"/>
+        <axis xyz="0 0 -1"/>
+    </joint>
+    <link name="wheel_2">
+        <visual>
+            <geometry>
+                <cylinder length="0.038" radius="0.05" />/>
+            </geometry>
+            <material name="blue"/>
+        </visual>
+    </link>
+    <!-- REAR LEFT WHEEL AKA wheel_3 -->
+    <joint name="wheel_3_joint" type="continuous">
+        <parent link="base_link"/>
+        <child link="wheel_3"/>
+        <origin xyz="-0.1575 0.1575 0" rpy="-${pi/2} 0 ${pi/4}"/>
+        <axis xyz="0 0 1"/>
+    </joint>
+    <link name="wheel_3">
+        <visual>
+            <geometry>
+                <cylinder length="0.038" radius="0.05" />/>
+            </geometry>
+            <material name="blue"/>
+        </visual>
+    </link>
+    <!-- REAR RIGHT WHEEL AKA wheel_4 -->
+    <joint name="wheel_4_joint" type="continuous">
+        <parent link="base_link"/>
+        <child link="wheel_4"/>
+        <origin xyz="-0.1575 -0.1575 0" rpy="${pi/2} 0 -${pi/4}"/>
+        <axis xyz="0 0 -1"/>
+    </joint>
+    <link name="wheel_4">
+        <visual>
+            <geometry>
+                <cylinder length="0.038" radius="0.05" />/>
             </geometry>
             <material name="blue"/>

Commit message: added collision and inertial for chassis & wheels

File: description/robot_core.xacro (robot description, xacro)
@@ -1,4 +1,5 @@
 <?xml version="1.0"?>
 <robot xmlns:xacro="http://www.ros.org/wiki/xacro">
+    <xacro:include filename="inertial_macros.xacro"/>
     <!-- links and joints go here -->
     <!-- The rest of the robot can be described from base_link, which is the centre point of the four driving wheels -->
@@ -21,4 +22,14 @@
             <material name="white"/>
         </visual>
+        <!-- physics model -->
+        <collision>
+            <origin xyz="0 0 0.75" rpy="0 0 0"/>
+            <geometry>
+                <box size="0.54 0.54 1.5"/>
+            </geometry>
+        </collision>
+        <xacro:inertial_box mass="10" x="0.54" y="0.54" z="1.5">
+            <origin xyz="0 0 0.75" rpy="0 0 0"/>
+        </xacro:inertial_box>
     </link>
     <!-- FRONT LEFT WHEEL AKA wheel_1 -->
@@ -32,8 +43,16 @@
         <visual>
             <geometry>
-                <cylinder length="0.038" radius="0.05" />/>
+                <cylinder length="0.038" radius="0.05" />
             </geometry>
             <material name="blue"/>
         </visual>
+        <collision>
+            <geometry>
+                <cylinder length="0.038" radius="0.05" />
+            </geometry>
+        </collision>
+        <xacro:inertial_cylinder mass="0.2" length="0.038" radius="0.05">
+            <origin xyz="0 0 0" rpy="0 0 0"/>
+        </xacro:inertial_cylinder>
     </link>
     <!-- FRONT RIGHT WHEEL AKA wheel_2 -->
@@ -47,8 +66,16 @@
         <visual>
             <geometry>
-                <cylinder length="0.038" radius="0.05" />/>
+                <cylinder length="0.038" radius="0.05" />
             </geometry>
             <material name="blue"/>
         </visual>
+        <collision>
+            <geometry>
+                <cylinder length="0.038" radius="0.05" />
+            </geometry>
+        </collision>
+        <xacro:inertial_cylinder mass="0.2" length="0.038" radius="0.05">
+            <origin xyz="0 0 0" rpy="0 0 0"/>
+        </xacro:inertial_cylinder>
     </link>
     <!-- REAR LEFT WHEEL AKA wheel_3 -->
@@ -62,8 +89,16 @@
         <visual>
             <geometry>
-                <cylinder length="0.038" radius="0.05" />/>
+                <cylinder length="0.038" radius="0.05" />
             </geometry>
             <material name="blue"/>
         </visual>
+        <collision>
+            <geometry>
+                <cylinder length="0.038" radius="0.05" />
+            </geometry>
+        </collision>
+        <xacro:inertial_cylinder mass="0.2" length="0.038" radius="0.05">
+            <origin xyz="0 0 0" rpy="0 0 0"/>
+        </xacro:inertial_cylinder>
     </link>
     <!-- REAR RIGHT WHEEL AKA wheel_4 -->
@@ -77,8 +112,16 @@
         <visual>
             <geometry>
-                <cylinder length="0.038" radius="0.05" />/>
+                <cylinder length="0.038" radius="0.05" />
             </geometry>
             <material name="blue"/>
         </visual>
+        <collision>
+            <geometry>
+                <cylinder length="0.038" radius="0.05" />
+            </geometry>
+        </collision>
+        <xacro:inertial_cylinder mass="0.2" length="0.038" radius="0.05">
+            <origin xyz="0 0 0" rpy="0 0 0"/>
+        </xacro:inertial_cylinder>
     </link>
 </robot>

Commit message: updated instructions and included gazebo color

File: description/robot_core.xacro (robot description, xacro)
@@ -33,4 +33,8 @@
         </xacro:inertial_box>
     </link>
+    <!-- gazebo specific description -->
+    <gazebo reference="chassis">
+        <material>Gazebo/White</material>
+    </gazebo>
     <!-- FRONT LEFT WHEEL AKA wheel_1 -->
     <joint name="wheel_1_joint" type="continuous">
@@ -56,4 +60,7 @@
         </xacro:inertial_cylinder>
     </link>
+    <gazebo reference="wheel_1">
+        <material>Gazebo/Blue</material>
+    </gazebo>
     <!-- FRONT RIGHT WHEEL AKA wheel_2 -->
     <joint name="wheel_2_joint" type="continuous">
@@ -79,4 +86,7 @@
         </xacro:inertial_cylinder>
     </link>
+    <gazebo reference="wheel_2">
+        <material>Gazebo/Blue</material>
+    </gazebo>
     <!-- REAR LEFT WHEEL AKA wheel_3 -->
     <joint name="wheel_3_joint" type="continuous">
@@ -102,4 +112,7 @@
         </xacro:inertial_cylinder>
     </link>
+    <gazebo reference="wheel_3">
+        <material>Gazebo/Blue</material>
+    </gazebo>
     <!-- REAR RIGHT WHEEL AKA wheel_4 -->
     <joint name="wheel_4_joint" type="continuous">
@@ -125,3 +138,6 @@
         </xacro:inertial_cylinder>
     </link>
+    <gazebo reference="wheel_4">
+        <material>Gazebo/Blue</material>
+    </gazebo>
 </robot>

Commit message: added frame model for rviz
gazebo not functional yet

File: description/robot_core.xacro (robot description, xacro)
@@ -16,7 +16,9 @@
         <visual>
             <!-- by default, the origin is centred around the link origin, so offset it by half the height -->
-            <origin xyz="0 0 0.75" rpy="0 0 0"/>
+            <!-- <origin xyz="0 0 0.75" rpy="0 0 0"/> -->
             <geometry>
-                <box size="0.54 0.54 1.5"/>
+                <!-- <box size="0.54 0.54 1.5"/> -->
+                <mesh filename="package://robocock/meshes/frame_ultra_low_poly.stl"/>
+                <!-- <mesh filename="model://frame_ultra_low_poly.stl"/> -->
             </geometry>
             <material name="white"/>
